Commit message: prep for planning testing

File: src/handover_description/urdf/ur5e.xacro (robot description, xacro)
@@ -4,4 +4,10 @@
     <material name="gripper_light_blue">
         <color rgba="0.55 0.75 0.95 1.0"/>
+    </material>
+    <material name="tool_orange">
+        <color rgba="0.9 0.5 0.1 1.0"/>
+    </material>
+    <material name="tool_grey">
+        <color rgba="0.5 0.5 0.5 1.0"/>
     </material>
     <!-- UR5e arm with a simple cylindrical gripper and a TCP frame at the gripper tip -->
@@ -56,4 +62,29 @@
         </joint>
         <link name="${tf_prefix}tcp"/>
+        <link name="${tf_prefix}held_tool">
+            <visual>
+                <origin xyz="0 0 0.05" rpy="0 0 0"/>
+                <geometry><cylinder radius="0.015" length="0.10"/></geometry>
+                <material name="tool_orange"/>
+            </visual>
+            <collision>
+                <origin xyz="0 0 0.05" rpy="0 0 0"/>
+                <geometry><cylinder radius="0.015" length="0.10"/></geometry>
+            </collision>
+            <visual>
+                <origin xyz="0 0 -0.05" rpy="0 0 0"/>
+                <geometry><cylinder radius="0.005" length="0.10"/></geometry>
+                <material name="tool_grey"/>
+            </visual>
+            <collision>
+                <origin xyz="0 0 -0.05" rpy="0 0 0"/>
+                <geometry><cylinder radius="0.005" length="0.10"/></geometry>
+            </collision>
+            <inertial>
+                <mass value="0.15"/>
+                <inertia ixx="0.000504" iyy="0.000504" izz="0.0000075"
+                        ixy="0" ixz="0" iyz="0"/>
+            </inertial>
+        </link>
         <joint name="${tf_prefix}gripper_to_tcp" type="fixed">
             <parent link="${tf_prefix}gripper"/>
@@ -61,4 +92,9 @@
             <origin xyz="0 0 ${gripper_length}" rpy="0 0 0"/>
         </joint>
+        <joint name="${tf_prefix}tcp_to_held_tool" type="fixed">
+            <parent link="${tf_prefix}tcp"/>
+            <child link="${tf_prefix}held_tool"/>
+            <origin xyz="0 -0.05 0.005" rpy="1.5708 0 0"/>
+        </joint>
     </xacro:macro>
 </robot>
